File: GYRO_PCB/GYRO_PCB.kicad_pcb (KiCad board)
At the start: 2 copper layers, 4 parts, among them J1 Pmod GYRO, J2 FLASH Socket 1, J3 FLASH Socket 2, U1 NUCLEO64-F446RE

Commit message: feat: finish PCB draft
Parts:
- added C1: 0.1uF, Capacitor_THT:C_Disc_D8.0mm_W2.5mm_P5.00mm, F.Cu at (144.6, 82.4)
- added G***: LOGO, FOOTPRINTS:logo, F.Cu at (131.7, 95.1)
- added H1: MountingHole, MountingHole:MountingHole_2.2mm_M2_ISO14580, F.Cu at (111.6, 77.8)
- added H2: MountingHole, MountingHole:MountingHole_2.2mm_M2_ISO14580, F.Cu at (179.4, 77.8)
- added H3: MountingHole, MountingHole:MountingHole_2.2mm_M2_ISO14580, F.Cu at (111.5, 130.4)
- added H4: MountingHole, MountingHole:MountingHole_2.2mm_M2_ISO14580, F.Cu at (179.4, 130.4)
- added J4: Power Terminal, TerminalBlock_MetzConnect:TerminalBlock_MetzConnect_Type011_RT05503HBLC_1x03_P5.00mm_Horizontal, F.Cu at (139.1, 82.4)
- added R1: 100k, Resistor_THT:R_Axial_DIN0207_L6.3mm_D2.5mm_P10.16mm_Horizontal, F.Cu at (129.6, 102.8)
- added R2: 100k, Resistor_THT:R_Axial_DIN0207_L6.3mm_D2.5mm_P10.16mm_Horizontal, F.Cu at (129.6, 107.9)
- added R3: 100k, Resistor_THT:R_Axial_DIN0207_L6.3mm_D2.5mm_P10.16mm_Horizontal, F.Cu at (156.4, 120.6)
- added R4: 10k, Resistor_THT:R_Axial_DIN0207_L6.3mm_D2.5mm_P10.16mm_Horizontal, F.Cu at (140.0, 118.0)
- added R5: 10k, Resistor_THT:R_Axial_DIN0207_L6.3mm_D2.5mm_P10.16mm_Horizontal, F.Cu at (140.1, 123.0)
- added R6: 10k, Resistor_THT:R_Axial_DIN0207_L6.3mm_D2.5mm_P10.16mm_Horizontal, F.Cu at (153.5, 96.3)
- added R7: 10k, Resistor_THT:R_Axial_DIN0207_L6.3mm_D2.5mm_P10.16mm_Horizontal, F.Cu at (139.3, 96.3)
- moved J2 44.4 mm to (148.4, 102.8)
- moved J3 42.6 mm to (163.6, 102.8)
- moved U1 18.2 mm to (145.5, 91.0)
- moved J1 15.6 mm to (155.5, 82.0), turned to 90 degrees
Connections:
- J1 pad 7: unconnected-(J1-GND-Pad7) -> GND
- J1 pad 8: unconnected-(J1-VCC-Pad8) -> +3V3
- U1 pad CN6_6: (no net) -> GND
- U1 pad CN6_7: (no net) -> GND
- U1 pad CN7_6: (no net) -> NUCLEO_E5V
- U1 pad CN8_3: (no net) -> NUCLEO_FLASH_CS
Routing:
- net NUCLEO_FLASH_SPI2_MISO: track 0.00 -> 43.8 mm
- net NUCLEO_FLASH_SPI2_MOSI: track 0.00 -> 34.3 mm
- net NUCLEO_E5V: track 0.00 -> 19.5 mm
- net NUCLEO_FLASH_SCLK: track 0.00 -> 12.5 mm
- net NUCLEO_GYRO_I2C1_SDA: track 0.00 -> 9.73 mm
- net Net-(J2-DQ3/HOLD#): track 0.00 -> 8.67 mm
- net Net-(J2-RESET#): track 0.00 -> 8.66 mm
- net NUCLEO_FLASH_CS: track 0.00 -> 8.38 mm
- net Net-(J3-W#/DQ2): track 0.00 -> 7.23 mm
- net NUCLEO_GYRO_I2C1_SCL: track 0.00 -> 6.13 mm
Other:
- board outline added: 72.4 x 57.2 mm
- board text added: "1"
- board text added: "3V3"
- board text added: "5V"
- board text added: "Flash Socket"
- board text added: "GND"
- board text added: "github.com/fectec/CUKET_GyroscopeShield"
